File: ExospineV2/ExospineV2.kicad_sch (KiCad schematic)
At the start: 6 parts, among them J1 GPIO, U1 CAT24C256

Commit message: ajout
Parts:
- added J2, J4: Conn_01x03_Socket, Connector_JST:JST_EH_B3B-EH-A_1x03_P2.50mm_Vertical, symbol Connector:Conn_01x03_Socket
- added J3: Conn_01x08_Socket, Connector_JST:JST_EH_S8B-EH_1x08_P2.50mm_Horizontal, symbol Connector:Conn_01x08_Socket
- added R3: 4.7k, Resistor_SMD:R_0402_1005Metric, symbol Device:R
Connections:
- net +3V3: now also J4.1 (Pin_1), R3.1
- net GND: now also J4.3 (Pin_3)
- new net GPIO17/SDA1: J4.2 (Pin_2), R3.2
Other:
- note added: "Thermistances"
Changed lines of the file:
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@@
   (junction (at 76.2 68.58) (diameter 1.016) (color 0 0 0 0)
+  )
+  (junction (at 147.32 46.99) (diameter 0) (color 0 0 0 0)
+  )
+  (junction (at 147.32 38.1) (diameter 0) (color 0 0 0 0)
   )
   (junction (at 76.2 63.5) (diameter 1.016) (color 0 0 0 0)
@@
     (stroke (width 0) (type solid))
   )
+  (wire (pts (xy 147.32 38.1) (xy 147.32 39.37))
+    (stroke (width 0) (type default))
+  )
+  (wire (pts (xy 147.32 46.99) (xy 154.94 46.99))
+    (stroke (width 0) (type default))
+  )
   (wire (pts (xy 58.42 38.1) (xy 60.96 38.1))
     (stroke (width 0) (type solid))
@@
     (stroke (width 0) (type solid))
   )
+  (wire (pts (xy 134.62 52.07) (xy 160.02 52.07))
+    (stroke (width 0) (type default))
+  )
   (wire (pts (xy 73.66 76.2) (xy 100.33 76.2))
     (stroke (width 0) (type solid))
@@
     (stroke (width 0) (type solid))
   )
+  (wire (pts (xy 134.62 38.1) (xy 147.32 38.1))
+    (stroke (width 0) (type default))
+  )
   (wire (pts (xy 31.75 33.02) (xy 60.96 33.02))
     (stroke (width 0) (type solid))
@@
     (stroke (width 0) (type solid))
   )
+  (wire (pts (xy 154.94 40.64) (xy 154.94 46.99))
+    (stroke (width 0) (type default))
+  )
   (wire (pts (xy 31.75 35.56) (xy 60.96 35.56))
     (stroke (width 0) (type solid))
@@
     (stroke (width 0) (type solid))
   )
+  (wire (pts (xy 147.32 46.99) (xy 147.32 49.53))
+    (stroke (width 0) (type default))
+  )
   (wire (pts (xy 31.75 66.04) (xy 60.96 66.04))
     (stroke (width 0) (type solid))
@@
     (stroke (width 0) (type solid))
   )
+  (wire (pts (xy 147.32 38.1) (xy 160.02 38.1))
+    (stroke (width 0) (type default))
+  )
+  (wire (pts (xy 160.02 43.18) (xy 160.02 52.07))
+    (stroke (width 0) (type default))
+  )
   (wire (pts (xy 73.66 73.66) (xy 100.33 73.66))
     (stroke (width 0) (type solid))
@@
     (stroke (width 0) (type solid))
   )
+  (wire (pts (xy 160.02 40.64) (xy 154.94 40.64))
+    (stroke (width 0) (type default))
+  )
   (wire (pts (xy 67.31 165.1) (xy 67.31 175.26))
     (stroke (width 0) (type solid))
@@
     (stroke (width 0) (type solid))
   )
+  (wire (pts (xy 132.08 49.53) (xy 147.32 49.53))
+    (stroke (width 0) (type default))
+  )
   (wire (pts (xy 76.2 68.58) (xy 76.2 80.01))
     (stroke (width 0) (type solid))
@@
   (wire (pts (xy 73.66 60.96) (xy 100.33 60.96))
     (stroke (width 0) (type solid))
+  )
+  (text "Thermistances\n" (at 143.51 30.48 0)
+    (effects (font (size 1.27 1.27)) (justify left bottom))
   )
   (text "Additional pin functions:\nhttps://pinout.xyz/" (at 179.07 180.34 0)
@@
   (label "GPIO23" (at 100.33 45.72 180) (fields_autoplaced)
     (effects (font (size 1.27 1.27)) (justify right bottom))
+  )
+  (label "GPIO17{slash}SDA1" (at 132.08 49.53 0) (fields_autoplaced)
+    (effects (font (size 1.27 1.27)) (justify left bottom))
   )
   (label "GPIO4{slash}GPCLK0" (at 31.75 35.56 0) (fields_autoplaced)
@@
     )
   )
+  (symbol (lib_id "Connector:Conn_01x03_Socket") (at 165.1 40.64 0) (unit 1)
+    (in_bom yes) (on_board yes) (dnp no) (fields_autoplaced)
+    (property "Reference" "J4" (at 166.37 39.37 0)
+      (effects (font (size 1.27 1.27)) (justify left))
+    )
+    (property "Value" "Conn_01x03_Socket" (at 166.37 41.91 0)
+      (effects (font (size 1.27 1.27)) (justify left))
+    )
+    (property "Footprint" "Connector_JST:JST_EH_B3B-EH-A_1x03_P2.50mm_Vertical" (at 165.1 40.64 0)
+      (effects (font (size 1.27 1.27)) hide)
+    )
+    (property "Datasheet" "~" (at 165.1 40.64 0)
+      (effects (font (size 1.27 1.27)) hide)
+    )
+    (pin "1")
+    (pin "2")
+    (pin "3")
+    (instances
+      (project "ExospineV2"
+        (path "/e63e39d7-6ac0-4ffd-8aa3-1841a4541b55"
+          (reference "J4") (unit 1)
+        )
+      )
+    )
+  )
   (symbol (lib_id "Device:R_Small") (at 93.98 170.18 0) (unit 1)
     (in_bom yes) (on_board yes) (dnp no)
@@
     )
   )
+  (symbol (lib_name "GND_1") (lib_id "power:GND") (at 134.62 52.07 0) (unit 1)
+    (in_bom yes) (on_board yes) (dnp no) (fields_autoplaced)
+    (property "Reference" "#PWR05" (at 134.62 58.42 0)
+      (effects (font (size 1.27 1.27)) hide)
+    )
+    (property "Value" "GND" (at 134.62 57.15 0)
+      (effects (font (size 1.27 1.27)))
+    )
+    (property "Footprint" "" (at 134.62 52.07 0)
+      (effects (font (size 1.27 1.27)) hide)
+    )
+    (property "Datasheet" "" (at 134.62 52.07 0)
+      (effects (font (size 1.27 1.27)) hide)
+    )
+    (pin "1")
+    (instances
+      (project "ExospineV2"
+        (path "/e63e39d7-6ac0-4ffd-8aa3-1841a4541b55"
+          (reference "#PWR05") (unit 1)
+        )
+      )
+    )
+  )
   (symbol (lib_id "power:+3.3V") (at 101.6 162.56 0) (unit 1)
     (in_bom yes) (on_board yes) (dnp no)
@@
         (path "/e63e39d7-6ac0-4ffd-8aa3-1841a4541b55"
           (reference "#PWR0101") (unit 1)
+        )
+      )
+    )
+  )
+  (symbol (lib_id "Device:R") (at 147.32 43.18 0) (unit 1)
+    (in_bom yes) (on_board yes) (dnp no) (fields_autoplaced)
+    (property "Reference" "R3" (at 149.86 41.91 0)
+      (effects (font (size 1.27 1.27)) (justify left))
+    )
+    (property "Value" "4.7k" (at 149.86 44.45 0)
+      (effects (font (size 1.27 1.27)) (justify left))
+    )
+    (property "Footprint" "Resistor_SMD:R_0402_1005Metric" (at 145.542 43.18 90)
+      (effects (font (size 1.27 1.27)) hide)
+    )
+    (property "Datasheet" "~" (at 147.32 43.18 0)
+      (effects (font (size 1.27 1.27)) hide)
+    )
+    (pin "1")
+    (pin "2")
+    (instances
+      (project "ExospineV2"
+        (path "/e63e39d7-6ac0-4ffd-8aa3-1841a4541b55"
+          (reference "R3") (unit 1)
         )
       )
@@
     )
   )
+  (symbol (lib_id "power:+3.3V") (at 134.62 38.1 0) (unit 1)
+    (in_bom yes) (on_board yes) (dnp no)
+    (property "Reference" "#PWR06" (at 134.62 41.91 0)
+      (effects (font (size 1.27 1.27)) hide)
+    )
+    (property "Value" "+3.3V" (at 134.9883 33.7756 0)
+      (effects (font (size 1.27 1.27)))
+    )
+    (property "Footprint" "" (at 134.62 38.1 0)
+      (effects (font (size 1.27 1.27)))
+    )
+    (property "Datasheet" "" (at 134.62 38.1 0)
+      (effects (font (size 1.27 1.27)))
+    )
+    (pin "1")
+    (instances
+      (project "ExospineV2"
+        (path "/e63e39d7-6ac0-4ffd-8aa3-1841a4541b55"
+          (reference "#PWR06") (unit 1)
+        )
+      )
+    )
+  )
+  (symbol (lib_id "Connector:Conn_01x08_Socket") (at 195.58 71.12 0) (unit 1)
+    (in_bom yes) (on_board yes) (dnp no) (fields_autoplaced)
+    (property "Reference" "J3" (at 196.85 71.12 0)
+      (effects (font (size 1.27 1.27)) (justify left))
+    )
+    (property "Value" "Conn_01x08_Socket" (at 196.85 73.66 0)
+      (effects (font (size 1.27 1.27)) (justify left))
+    )
+    (property "Footprint" "Connector_JST:JST_EH_S8B-EH_1x08_P2.50mm_Horizontal" (at 195.58 71.12 0)
+      (effects (font (size 1.27 1.27)) hide)
+    )
+    (property "Datasheet" "~" (at 195.58 71.12 0)
+      (effects (font (size 1.27 1.27)) hide)
+    )
+    (pin "1")
+    (pin "2")
+    (pin "3")
+    (pin "4")
+    (pin "5")
+    (pin "6")
+    (pin "7")
+    (pin "8")
+    (instances
+      (project "ExospineV2"
+        (path "/e63e39d7-6ac0-4ffd-8aa3-1841a4541b55"
+          (reference "J3") (unit 1)
+        )
+      )
+    )
+  )
   (symbol (lib_id "power:GND") (at 81.28 190.5 0) (unit 1)
     (in_bom yes) (on_board yes) (dnp no)
@@
         )
       )
+    )
+  )
+  (symbol (lib_id "Connector:Conn_01x03_Socket") (at 194.31 52.07 0) (unit 1)
+    (in_bom yes) (on_board yes) (dnp no) (fields_autoplaced)
+    (property "Reference" "J2" (at 195.58 50.8 0)
+      (effects (font (size 1.27 1.27)) (justify left))
+    )
+    (property "Value" "Conn_01x03_Socket" (at 195.58 53.34 0)
+      (effects (font (size 1.27 1.27)) (justify left))
+    )
+    (property "Footprint" "Connector_JST:JST_EH_B3B-EH-A_1x03_P2.50mm_Vertical" (at 194.31 52.07 0)
+      (effects (font (size 1.27 1.27)) hide)
+    )
+    (property "Datasheet" "~" (at 194.31 52.07 0)
+      (effects (font (size 1.27 1.27)) hide)
+    )
+    (pin "1")
+    (pin "2")
+    (pin "3")
+    (instances
+      (project "ExospineV2"
+        (path "/e63e39d7-6ac0-4ffd-8aa3-1841a4541b55"
+          (reference "J2") (unit 1)
+        )
+      )
