File: ExospineV2.kicad_sch (KiCad schematic)
At the start: 2 parts, among them U1 RASPBERRY_PI_4B_4GB

Commit message: Move files
Parts:
- removed R1: 10k, Resistor_SMD:R_0603_1608Metric, symbol Device:R
- removed U1: RASPBERRY_PI_4B_4GB, RASPBERRY_PI_4B_4GB:MODULE_RASPBERRY_PI_4B_4GB, symbol RASPBERRY_PI_4B_4GB:RASPBERRY_PI_4B_4GB
- added C1: 100n, symbol Device:C_Small
- added J1: GPIO, Connector_PinSocket_2.54mm:PinSocket_2x20_P2.54mm_Vertical, symbol Connector_Generic:Conn_02x20_Odd_Even
- added J2, J4: Conn_01x03_Socket, Connector_JST:JST_EH_B3B-EH-A_1x03_P2.50mm_Vertical, symbol Connector:Conn_01x03_Socket
- added J3: Conn_01x08_Socket, Connector_JST:JST_EH_S8B-EH_1x08_P2.50mm_Horizontal, symbol Connector:Conn_01x08_Socket
- added JP1: ID_WP, symbol Jumper:SolderJumper_2_Open
- added R1, R2: 3.9k, symbol Device:R_Small
- added R3: 4.7k, Resistor_SMD:R_0402_1005Metric, symbol Device:R
- added U1: CAT24C256, symbol Memory_EEPROM:CAT24C256
Connections:
- net GND: now also C1.2, J1.14 (Pin_14), J1.20 (Pin_20), J1.25 (Pin_25), J1.30 (Pin_30), J1.34 (Pin_34), J1.39 (Pin_39), J1.6 (Pin_6), J1.9 (Pin_9), J4.3 (Pin_3), U1.4 (GND)
- net GPIO14/TXD0: now also J1.8 (Pin_8)
- net GPIO15/RXD0: now also J1.10 (Pin_10)
- net GPIO16: now also J1.36 (Pin_36)
- net GPIO26: now also J1.37 (Pin_37)
- net GPIO2/SDA1: now also J1.3 (Pin_3)
- net GPIO3/SCL1: now also J1.5 (Pin_5)
- net GPIO5: now also J1.29 (Pin_29)
- net GPIO6: now also J1.31 (Pin_31)
- new net: JP1.1 (A), U1.7 (WP)
- new net +3V3: C1.1, J1.1 (Pin_1), J1.17 (Pin_17), J4.1 (Pin_1), JP1.2 (B), R1.1, R2.1, R3.1, U1.8 (VCC)
- new net +5V: J1.2 (Pin_2), J1.4 (Pin_4)
- new net GPIO10/SPI0.MOSI: J1.19 (Pin_19)
- new net GPIO11/SPI0.SCLK: J1.23 (Pin_23)
- new net GPIO12/PWM0: J1.32 (Pin_32)
- new net GPIO13/PWM1: J1.33 (Pin_33)
- new net GPIO17: J1.11 (Pin_11)
- new net GPIO17/SDA1: J4.2 (Pin_2), R3.2
- new net GPIO18/PCM.CLK: J1.12 (Pin_12)
- new net GPIO19/PCM.FS: J1.35 (Pin_35)
- new net GPIO20/PCM.DIN: J1.38 (Pin_38)
- new net GPIO21/PCM.DOUT: J1.40 (Pin_40)
- new net GPIO22: J1.15 (Pin_15)
- new net GPIO23: J1.16 (Pin_16)
- new net GPIO24: J1.18 (Pin_18)
- new net GPIO25: J1.22 (Pin_22)
- new net GPIO27: J1.13 (Pin_13)
- new net GPIO4/GPCLK0: J1.7 (Pin_7)
- new net GPIO7/SPI0.CE1: J1.26 (Pin_26)
- new net GPIO8/SPI0.CE0: J1.24 (Pin_24)
- new net GPIO9/SPI0.MISO: J1.21 (Pin_21)
- new net ID_SCL: J1.28 (Pin_28), R2.2, U1.6 (SCL)
- new net ID_SDA: J1.27 (Pin_27), R1.2, U1.5 (SDA)
- no-connect marks 0 -> 3
Other:
- note added: "Additional pin functions: https://pinout.xyz/"
- note added: "ID_SD and ID_SC PINS: These pins are reserved for HAT ID EEPROM. At boot time this I2C interface will be interrogated to look for an EEPROM that identifes the attached board and allows automagic setup of the GPIOs (and optionally, Linux drivers). Bridging JP1 enables write protection. DO NOT USE these pins for anything other than attaching an I2C ID EEPROM. Leave unconnected if ID EEPROM not requ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"
- note added: "Thermistances"
